File: driver_v1/driver_v1.kicad_sch (KiCad schematic)
At the start: 90 parts, among them J1 PMT, J2 SMA, J4 USB_B, Q1 MMBT2222A, Q2 MMBT2222A, T1 FL2015-9L, U1 ADP1613, U2 OPA314AIDBV, U3 ADA4891-1, U4 TPS7A2045PDBVR

Commit message: Include screws in BOM, add serial number location
Parts:
- H1, H2, H3, H4, H5: now in the parts list
Changed lines of the file:
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@@
 		(unit 1)
 		(exclude_from_sim yes)
-		(in_bom no)
+		(in_bom yes)
 		(on_board yes)
 		(dnp no)
@@
 		(unit 1)
 		(exclude_from_sim yes)
-		(in_bom no)
+		(in_bom yes)
 		(on_board yes)
 		(dnp no)
@@
 		(unit 1)
 		(exclude_from_sim yes)
-		(in_bom no)
+		(in_bom yes)
 		(on_board yes)
 		(dnp no)
@@
 		(unit 1)
 		(exclude_from_sim yes)
-		(in_bom no)
+		(in_bom yes)
 		(on_board yes)
 		(dnp no)
@@
 		(unit 1)
 		(exclude_from_sim yes)
-		(in_bom no)
+		(in_bom yes)
 		(on_board yes)
 		(dnp no)
